File: kicad/potenciostato.kicad_pcb (KiCad board)
At the start: 2 copper layers, 150 x 100 mm, 51 parts, among them J1 Conn_01x03_Female, J2 USB_B_Micro, J3 Conn_01x03_Male, U1 OP77, U2 TL082, U3 OP77, U4 OP77, U5 4016, U6 4016, U7 TL064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

Commit message: Actualicé los valores en PCB
Parts:
- R1: value R -> 15K
- R10, R11, R14, R16, R20, R21, R25, R27, R4, R6, R7: value R -> 1K
- R12, R17, R8: value R -> 3K3
- R13, R18, R9: value R -> 4K7
- R15, R19, R22, R23, R24, R26: value R -> 10K
- R2, R3: value 100k -> 100K
- R5: value R -> 1M
- RV10, RV11, RV12, RV3, RV6, RV7, RV8, RV9: value R_POT -> 1K
Connections:
- J2 pad 1: (no net) -> Net-(J2-Pad1)
- J2 pad 4: (no net) -> Net-(J2-Pad4)
- LPC1 pad 10: (no net) -> Net-(LPC1-Pad10)
- LPC1 pad 11: (no net) -> Net-(LPC1-Pad11)
- LPC1 pad 12: (no net) -> Net-(LPC1-Pad12)
- LPC1 pad 13: (no net) -> Net-(LPC1-Pad13)
- LPC1 pad 14: (no net) -> Net-(LPC1-Pad14)
- LPC1 pad 17: (no net) -> Net-(LPC1-Pad17)
- LPC1 pad 19: (no net) -> Net-(LPC1-Pad19)
- LPC1 pad 2: (no net) -> /LPC/5V
- LPC1 pad 20: (no net) -> Net-(LPC1-Pad20)
- LPC1 pad 25: (no net) -> Net-(LPC1-Pad25)
- LPC1 pad 26: (no net) -> Net-(LPC1-Pad26)
- LPC1 pad 27: (no net) -> Net-(LPC1-Pad27)
- LPC1 pad 28: (no net) -> /LPC/3.3V
- LPC1 pad 29: (no net) -> Net-(LPC1-Pad29)
- LPC1 pad 3: (no net) -> Net-(LPC1-Pad3)
- LPC1 pad 30: (no net) -> Net-(LPC1-Pad30)
- LPC1 pad 31: (no net) -> Net-(LPC1-Pad31)
- LPC1 pad 32: (no net) -> Net-(LPC1-Pad32)
- LPC1 pad 33: (no net) -> Net-(LPC1-Pad33)
- LPC1 pad 34: (no net) -> Net-(LPC1-Pad34)
- LPC1 pad 35: (no net) -> Net-(LPC1-Pad35)
- LPC1 pad 38: (no net) -> Net-(LPC1-Pad38)
- LPC1 pad 39: (no net) -> Net-(LPC1-Pad39)
- LPC1 pad 4: (no net) -> Net-(LPC1-Pad4)
- LPC1 pad 40: (no net) -> Net-(LPC1-Pad40)
- LPC1 pad 41: (no net) -> Net-(LPC1-Pad41)
- LPC1 pad 42: (no net) -> Net-(LPC1-Pad42)
- LPC1 pad 43: /LPC/P2.2 -> /LPC/P2.1
- LPC1 pad 44: /LPC/P2.1 -> /LPC/P2.2
- LPC1 pad 45: (no net) -> /salida_dac/OFF_DAC_1
- LPC1 pad 46: (no net) -> /salida_dac/OFF_DAC_2
- LPC1 pad 5: (no net) -> Net-(LPC1-Pad5)
- LPC1 pad 51: (no net) -> Net-(LPC1-Pad51)
- LPC1 pad 52: (no net) -> Net-(LPC1-Pad52)
- LPC1 pad 53: (no net) -> Net-(LPC1-Pad53)
- LPC1 pad 55: (no net) -> Net-(LPC1-Pad55)
- LPC1 pad 56: (no net) -> Net-(LPC1-Pad56)
- LPC1 pad 57: (no net) -> Net-(LPC1-Pad57)
- LPC1 pad 58: (no net) -> Net-(LPC1-Pad58)
- LPC1 pad 59: (no net) -> Net-(LPC1-Pad59)
- LPC1 pad 6: (no net) -> Net-(LPC1-Pad6)
- LPC1 pad 60: (no net) -> Net-(LPC1-Pad60)
- LPC1 pad 61: (no net) -> Net-(LPC1-Pad61)
- LPC1 pad 62: (no net) -> Net-(LPC1-Pad62)
- LPC1 pad 63: (no net) -> Net-(LPC1-Pad63)
- LPC1 pad 64: (no net) -> Net-(LPC1-Pad64)
- LPC1 pad 65: (no net) -> Net-(LPC1-Pad65)
- LPC1 pad 66: (no net) -> Net-(LPC1-Pad66)
- LPC1 pad 67: (no net) -> Net-(LPC1-Pad67)
- LPC1 pad 68: (no net) -> Net-(LPC1-Pad68)
- LPC1 pad 69: (no net) -> Net-(LPC1-Pad69)
- LPC1 pad 7: (no net) -> Net-(LPC1-Pad7)
- LPC1 pad 70: (no net) -> Net-(LPC1-Pad70)
- LPC1 pad 71: (no net) -> Net-(LPC1-Pad71)
- LPC1 pad 72: (no net) -> Net-(LPC1-Pad72)
- LPC1 pad 73: (no net) -> Net-(LPC1-Pad73)
- LPC1 pad 8: (no net) -> Net-(LPC1-Pad8)
- LPC1 pad 9: (no net) -> Net-(LPC1-Pad9)
- U1 pad 1: (no net) -> Net-(U1-Pad1)
- U1 pad 5: (no net) -> Net-(U1-Pad5)
- U1 pad 8: (no net) -> Net-(U1-Pad8)
- U3 pad 1: (no net) -> Net-(U3-Pad1)
- U3 pad 5: (no net) -> Net-(U3-Pad5)
- U3 pad 8: (no net) -> Net-(U3-Pad8)
- U4 pad 1: (no net) -> Net-(U4-Pad1)
- U4 pad 5: (no net) -> Net-(U4-Pad5)
- U4 pad 8: (no net) -> Net-(U4-Pad8)
- U6 pad 12: /salida_dac/OFF_I_2 -> /salida_dac/OFF_DAC_2
- U6 pad 6: /salida_dac/OFF_I_1 -> /salida_dac/OFF_DAC_1

Commit message: modificaciones finales al kickad
Parts:
- R10: value 1K -> 10K
- R23: value 10K -> 15K
- R25: value 1K -> 15K
