File: kicad/potenciostato.sch (KiCad schematic (older format))
At the start: 11 parts, among them J1 Conn_01x03_Female, J3 Conn_01x03_Male, U1 OP77, U2 TL082, U3 OP77, U4 OP77

Commit message: agregar identificador y comentarios a amplificadores
Other:
- note added: "Amplificador Tension Inversor\n(AMP I1)"
- note added: "Amplificador Tension Inversor\n(AMP T3)"
- note added: "Amplificador Transresistencia\n(AMP TR)"
Changed lines of the file:
@@
 EESchema Schematic File Version 4
 LIBS:potenciostato-cache
-EELAYER 26 0
+EELAYER 29 0
 EELAYER END
 $Descr A4 11693 8268
@@
 	-1   0    0    1
 $EndComp
+Text Notes 6950 5500 0    50   ~ 0
+Amplificador Transresistencia\n(AMP TR)
+Text Notes 4850 5500 0    50   ~ 0
+Amplificador Tension Inversor\n(AMP I1)
+Text Notes 6350 1700 0    50   ~ 0
+Amplificador Tension Inversor\n(AMP T3)
 $EndSCHEMATC

Commit message: agregada huella del lpc al pcb
Connections:
- wire segments 54 -> 71

Commit message: Modificaciones en schematic
Changed lines of the file:
@@
 EESchema Schematic File Version 4
-LIBS:potenciostato-cache
-EELAYER 26 0
+EELAYER 30 0
 EELAYER END
 $Descr A4 11693 8268
@@
 F1 "salida_dac.sch" 50
 F2 "DAC1" I L 3800 2250 50
-F3 "SW_FILTRO1" I L 3800 2650 50
-F4 "SW_FILTRO2" I L 3800 2750 50
+F3 "OFF_DAC_1" I L 3800 2650 50
+F4 "OFF_DAC_2" I L 3800 2750 50
 F5 "SW_GAIN1" I L 3800 2450 50
 F6 "SW_GAIN2" I L 3800 2550 50

Commit message: prueba
Parts:
- R1: value R -> 15K
- R2, R3: value 100k -> 100K
- R4: value R -> 1K
- R5: value R -> 1M
Changed lines of the file:
@@
 P 6600 2200
 F 0 "R2" V 6393 2200 50  0000 C CNN
-F 1 "100k" V 6484 2200 50  0000 C CNN
+F 1 "100K" V 6484 2200 50  0000 C CNN
 F 2 "Resistor_THT:R_Axial_DIN0207_L6.3mm_D2.5mm_P7.62mm_Horizontal" V 6530 2200 50  0001 C CNN
 F 3 "~" H 6600 2200 50  0001 C CNN
@@
 P 6950 2750
 F 0 "R3" V 6743 2750 50  0000 C CNN
-F 1 "100k" V 6834 2750 50  0000 C CNN
+F 1 "100K" V 6834 2750 50  0000 C CNN
 F 2 "Resistor_THT:R_Axial_DIN0207_L6.3mm_D2.5mm_P7.62mm_Horizontal" V 6880 2750 50  0001 C CNN
 F 3 "~" H 6950 2750 50  0001 C CNN
@@
 P 8000 4050
 F 0 "R5" V 7793 4050 50  0000 C CNN
-F 1 "R" V 7884 4050 50  0000 C CNN
+F 1 "1M" V 7884 4050 50  0000 C CNN
 F 2 "Resistor_THT:R_Axial_DIN0207_L6.3mm_D2.5mm_P7.62mm_Horizontal" V 7930 4050 50  0001 C CNN
 F 3 "~" H 8000 4050 50  0001 C CNN
@@
 P 6050 4200
 F 0 "R1" V 5843 4200 50  0000 C CNN
-F 1 "R" V 5934 4200 50  0000 C CNN
+F 1 "15K" V 5934 4200 50  0000 C CNN
 F 2 "Resistor_THT:R_Axial_DIN0207_L6.3mm_D2.5mm_P7.62mm_Horizontal" V 5980 4200 50  0001 C CNN
 F 3 "~" H 6050 4200 50  0001 C CNN
@@
 P 7100 4700
 F 0 "R4" V 6893 4700 50  0000 C CNN
-F 1 "R" V 6984 4700 50  0000 C CNN
+F 1 "1K" V 6984 4700 50  0000 C CNN
 F 2 "Resistor_THT:R_Axial_DIN0207_L6.3mm_D2.5mm_P7.62mm_Horizontal" V 7030 4700 50  0001 C CNN
 F 3 "~" H 7100 4700 50  0001 C CNN

Commit message: P2.6 a P2.7 en kicad, resuelto escalado de la señal en LPC
Parts:
- J1: symbol Connector:Conn_01x03_Female -> potenciostato-rescue:Conn_01x03_Female-Connector
- J3: symbol Connector:Conn_01x03_Male -> potenciostato-rescue:Conn_01x03_Male-Connector
- R1, R2, R3, R4, R5: symbol Device:R -> potenciostato-rescue:R-Device
- U1, U3, U4: symbol Amplifier_Operational:OP77 -> potenciostato-rescue:OP77-Amplifier_Operational
- U2: symbol Amplifier_Operational:TL082 -> potenciostato-rescue:TL082-Amplifier_Operational
Changed lines of the file:
@@
 $EndDescr
 $Comp
-L Amplifier_Operational:OP77 U4
+L potenciostato-rescue:OP77-Amplifier_Operational U4
 U 1 1 5CC24F96
 P 8300 4700
@@
 $EndComp
 $Comp
-L Device:R R2
+L potenciostato-rescue:R-Device R2
 U 1 1 5CC25964
 P 6600 2200
@@
 $EndComp
 $Comp
-L Device:R R3
+L potenciostato-rescue:R-Device R3
 U 1 1 5CC2629B
 P 6950 2750
@@
 $EndComp
 $Comp
-L Device:R R5
+L potenciostato-rescue:R-Device R5
 U 1 1 5CC26B83
 P 8000 4050
@@
 $EndComp
 $Comp
-L power:GND #PWR08
+L potenciostato-rescue:GND-power #PWR08
 U 1 1 5CC2AC7B
 P 8700 4900
@@
 	7500 4700 8000 4700
 $Comp
-L power:GND #PWR01
+L potenciostato-rescue:GND-power #PWR01
 U 1 1 5CD2A3FD
 P 1000 1100
@@
 $EndComp
 $Comp
-L Connector:Conn_01x03_Female J1
+L potenciostato-rescue:Conn_01x03_Female-Connector J1
 U 1 1 5CDF8979
 P 1850 1100
@@
 	7400 2400 7300 2400
 $Comp
-L power:GND #PWR07
+L potenciostato-rescue:GND-power #PWR07
 U 1 1 5CC2A149
 P 7300 2500
@@
 $EndComp
 $Comp
-L Connector:Conn_01x03_Male J3
+L potenciostato-rescue:Conn_01x03_Male-Connector J3
 U 1 1 5D250C0E
 P 9950 3350
@@
 Connection ~ 7950 3250
 $Comp
-L power:+5V #PWR02
+L potenciostato-rescue:+5V-power #PWR02
 U 1 1 5F8AF7F8
 P 1150 1000
@@
 $EndComp
 $Comp
-L power:-5V #PWR03
+L potenciostato-rescue:-5V-power #PWR03
 U 1 1 5F8AF868
 P 1150 1200
@@
 NoConn ~ 5700 7300
 $Comp
-L Amplifier_Operational:OP77 U1
+L potenciostato-rescue:OP77-Amplifier_Operational U1
 U 1 1 5F9FAD3E
 P 6200 4800
@@
 $EndComp
 $Comp
-L Device:R R1
+L potenciostato-rescue:R-Device R1
 U 1 1 5F9FAD44
 P 6050 4200
@@
 $EndComp
 $Comp
-L power:GND #PWR06
+L potenciostato-rescue:GND-power #PWR06
 U 1 1 5F9FAD4A
 P 6600 5000
@@
 	6600 4900 6600 5000
 $Comp
-L Device:R R4
+L potenciostato-rescue:R-Device R4
 U 1 1 5F9FD20A
 P 7100 4700
@@
 Connection ~ 5500 4200
 $Comp
-L Amplifier_Operational:TL082 U2
+L potenciostato-rescue:TL082-Amplifier_Operational U2
 U 1 1 601CBD2D
 P 8400 3250
@@
 $EndComp
 $Comp
-L Amplifier_Operational:TL082 U2
+L potenciostato-rescue:TL082-Amplifier_Operational U2
 U 2 1 601CBED5
 P 6350 3350
@@
 $EndComp
 $Comp
-L Amplifier_Operational:TL082 U2
+L potenciostato-rescue:TL082-Amplifier_Operational U2
 U 3 1 601CBFB9
 P 6550 3350
@@
 $EndComp
 $Comp
-L power:-5V #PWR0101
+L potenciostato-rescue:-5V-power #PWR0101
 U 1 1 601CC089
 P 6450 3650
@@
 $EndComp
 $Comp
-L power:+5V #PWR0102
+L potenciostato-rescue:+5V-power #PWR0102
 U 1 1 601CC0FC
 P 6450 3050
@@
 $EndComp
 $Comp
-L Amplifier_Operational:OP77 U3
+L potenciostato-rescue:OP77-Amplifier_Operational U3
 U 1 1 5CC225D1
 P 7700 2300
@@
 $EndComp
 $Comp
-L power:-5V #PWR0103
+L potenciostato-rescue:-5V-power #PWR0103
 U 1 1 601CC2C2
 P 6300 4500
@@
 $EndComp
 $Comp
-L power:-5V #PWR0104
+L potenciostato-rescue:-5V-power #PWR0104
 U 1 1 601CC383
 P 8400 4400
@@
 $EndComp
 $Comp
-L power:-5V #PWR0105
+L potenciostato-rescue:-5V-power #PWR0105
 U 1 1 601CC42A
 P 7600 2000
@@
 $EndComp
 $Comp
-L power:+5V #PWR0106
+L potenciostato-rescue:+5V-power #PWR0106
 U 1 1 601CC539
 P 7600 2600
@@
 $EndComp
 $Comp
-L power:+5V #PWR0107
+L potenciostato-rescue:+5V-power #PWR0107
 U 1 1 601CC592
 P 8400 5000
@@
 $EndComp
 $Comp
-L power:+5V #PWR0108
+L potenciostato-rescue:+5V-power #PWR0108
 U 1 1 601CC639
 P 6300 5100
@@
 	2050 3100 2050 3200
 $Comp
-L power:GND #PWR0130
+L potenciostato-rescue:GND-power #PWR0130
 U 1 1 609B9D8E
 P 2050 3200
