File: kicadv2/potenciostato.kicad_sch (KiCad schematic)
At the start: 28 parts, among them J10 Conn_01x01_Female, J11 Conn_01x01_Female, J12 Conn_01x01_Female, J3 Conn_01x03_Male, J4 Conn_01x01_Female, J5 Conn_01x01_Female, J6 Conn_01x01_Female, U1 OP77, U2 TL082, U3 OP77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

Commit message: simulaciones y kicad para placa nueva
Parts:
- removed R? (x3): 0K, Resistor_THT:R_Axial_DIN0207_L6.3mm_D2.5mm_P7.62mm_Horizontal, symbol potenciostato-rescue:R-Device
- removed RV? (x3): 1K, Potentiometer_THT:Potentiometer_Bourns_3266Y_Vertical, symbol salida_dac-rescue:R_POT-Device
- removed U? (x5): 4016, symbol 4xxx:4016
- added J1: Conn_01x03_Female, Connector:FanPinHeader_1x03_P2.54mm_Vertical, symbol potenciostato-rescue:Conn_01x03_Female-Connector
Connections:
- net +5V: now also J1.1 (Pin_1)
- net -5V: now also J1.3 (Pin_3)
- net GND: now also J1.2 (Pin_2)
- net at J3.1 (Pin_1), U4.2 (-): now also RV4.2, RV4.3; no longer R5.1
- net at R4.1, U4.6: now also R5.2; no longer RV4.1, RV4.2
- new net: R5.1, RV4.1
Other:
- removed sheet Fuente
- moved on the sheet: J10, J11, J12, J3, J4, J5, J6, R1, R2, R3, R4, R5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
