File: kicadv2/potenciostato.sch (KiCad schematic (older format))
At the start: 18 parts, among them J1 Conn_01x03_Female, J10 test_GND, J11 test_GND, J12 test_GND, J3 Conn_01x03_Male, J4 Conn_01x01_Female, J5 Conn_01x01_Female, J6 Conn_01x01_Female, U1 OP77, U2 TL082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

Commit message: se agrega 4316 y ganancia de corriente variable
Parts:
- removed J1: Conn_01x03_Female, Connector:FanPinHeader_1x03_P2.54mm_Vertical, symbol potenciostato-rescue:Conn_01x03_Female-Connector
- removed RV4: 1K, Potentiometer_THT:Potentiometer_Bourns_3266Y_Vertical, symbol salida_dac-rescue:R_POT-Device
- added C? (x4): 10uF, symbol potenciostato-rescue:CP-Device
- added C? (x2): C, symbol Device:C
- added D?: D_Bridge_+-AA, symbol Device:D_Bridge_+-AA
- added R?: 10K, Resistor_THT:R_Axial_DIN0207_L6.3mm_D2.5mm_P7.62mm_Horizontal, symbol potenciostato-rescue:R-Device
- added R?: 4K7, Resistor_THT:R_Axial_DIN0207_L6.3mm_D2.5mm_P7.62mm_Horizontal, symbol potenciostato-rescue:R-Device
- added R?: 100K, Resistor_THT:R_Axial_DIN0207_L6.3mm_D2.5mm_P7.62mm_Horizontal, symbol potenciostato-rescue:R-Device
- added TR?: ADT2-71T, RF_Mini-Circuits:Mini-Circuits_CD637_H5.23mm, symbol Transformer:ADT2-71T
- added U? (x5): 4316, symbol 4316:4316
- added U?: L7805, symbol Regulator_Linear:L7805
- added U?: L7905, symbol Regulator_Linear:L7905
- J4: value Conn_01x01_Female -> test_I
- J5: value Conn_01x01_Female -> test_V
- J6: value Conn_01x01_Female -> test_DAC
- R1: value 33K -> 1K
- R5: value 0K -> 6K8
Connections:
- wire segments 64 -> 142
Other:
- moved on the sheet: J10, J11, J12, J3, J4, J5, J6, R1, R2, R3, R4, R5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

Commit message: agregado lo de Hernan y fixeado el kicad pcb
Parts:
- C1, C2, C5, C6: renamed from C?; footprint (none) -> Capacitor_THT:CP_Radial_D5.0mm_P2.00mm
- C3, C4: renamed from C?; value C -> 100nF; footprint (none) -> Capacitor_SMD:C_1206_3216Metric_Pad1.33x1.80mm_HandSolder
- D1: renamed from D?; footprint (none) -> Diode_SMD:Diode_Bridge_Vishay_DFS
- J10, J11, J12, J4, J5, J6: footprint Connector_PinHeader_2.54mm:PinHeader_1x01_P2.54mm_Vertical -> Connector_PinHeader_1.00mm:PinHeader_1x01_P1.00mm_Vertical
- J3: footprint Connector:FanPinHeader_1x03_P2.54mm_Vertical -> Connector_Phoenix_MC:PhoenixContact_MCV_1,5_3-G-3.5_1x03_P3.50mm_Vertical
- R1, R2, R4, R5: footprint Resistor_THT:R_Axial_DIN0207_L6.3mm_D2.5mm_P7.62mm_Horizontal -> Resistor_SMD:R_1206_3216Metric_Pad1.30x1.75mm_HandSolder
- R11, R12, R15: renamed from R?; footprint Resistor_THT:R_Axial_DIN0207_L6.3mm_D2.5mm_P7.62mm_Horizontal -> Resistor_SMD:R_1206_3216Metric_Pad1.30x1.75mm_HandSolder
- R3: footprint Resistor_THT:R_Axial_DIN0207_L6.3mm_D2.5mm_P10.16mm_Horizontal -> Resistor_SMD:R_1206_3216Metric_Pad1.30x1.75mm_HandSolder
- U1, U3, U4: footprint Package_DIP:DIP-8_W7.62mm_LongPads -> Package_SO:HSOP-8-1EP_3.9x4.9mm_P1.27mm_EP2.41x3.1mm
- U5: renamed from U?; footprint (none) -> Package_DIP:DIP-16_W7.62mm_LongPads
- U6, U8: renamed from U?; footprint (none) -> Package_TO_SOT_THT:TO-220-3_Vertical
- gave numbers to parts that had none: 1
