File: kicadv2/potenciostato.kicad_pcb (KiCad board)
At the start: 2 copper layers, 100 x 100 mm, 57 parts, among them U1 OP77, U2 TL082, U3 OP77, U4 OP77, U5 4316, U6 L7805, U7 TL064, U8 L7905, U9 TL082

Commit message: trazado pdf kicad
Connections:
- U9 pad 5: Net-(R16-Pad1) -> GND
- U9 pad 6: GND -> Net-(R16-Pad1)
Routing:
- net GND: track 25.9 -> 32.7 mm
- net Net-(R16-Pad1): track 7.78 -> 6.72 mm
