File: kicad_reducido/salida_dac.sch (KiCad schematic (older format))
At the start: 22 parts, among them U7 TL064

Commit message: ruteado kicad reducido parcialmente completo
Parts:
- U7: footprint Package_DIP:DIP-14_W10.16mm_LongPads -> Package_DIP:DIP-14_W7.62mm_Socket_LongPads
Changed lines of the file:
@@
 F 0 "U7" H 4550 3250 50  0000 C CNN
 F 1 "TL064" H 4750 3050 50  0000 C CNN
-F 2 "Package_DIP:DIP-14_W10.16mm_LongPads" H 4450 3050 50  0001 C CNN
+F 2 "Package_DIP:DIP-14_W7.62mm_Socket_LongPads" H 4450 3050 50  0001 C CNN
 F 3 "http://www.ti.com/lit/ds/symlink/tl061.pdf" H 4550 3150 50  0001 C CNN
 	1    4500 2950
@@
 F 0 "U7" H 7800 4000 50  0000 C CNN
 F 1 "TL064" H 7800 3850 50  0000 C CNN
-F 2 "Package_DIP:DIP-14_W10.16mm_LongPads" H 7550 3850 50  0001 C CNN
+F 2 "Package_DIP:DIP-14_W7.62mm_Socket_LongPads" H 7550 3850 50  0001 C CNN
 F 3 "http://www.ti.com/lit/ds/symlink/tl061.pdf" H 7650 3950 50  0001 C CNN
 	2    7600 3750
@@
 F 0 "U7" H 2850 6667 50  0000 C CNN
 F 1 "TL064" H 2850 6576 50  0000 C CNN
-F 2 "Package_DIP:DIP-14_W10.16mm_LongPads" H 2800 6400 50  0001 C CNN
+F 2 "Package_DIP:DIP-14_W7.62mm_Socket_LongPads" H 2800 6400 50  0001 C CNN
 F 3 "http://www.ti.com/lit/ds/symlink/tl061.pdf" H 2900 6500 50  0001 C CNN
 	3    2850 6300
@@
 F 0 "U7" H 6350 5650 50  0000 C CNN
 F 1 "TL064" H 6300 5726 50  0000 C CNN
-F 2 "Package_DIP:DIP-14_W10.16mm_LongPads" H 6250 5550 50  0001 C CNN
+F 2 "Package_DIP:DIP-14_W7.62mm_Socket_LongPads" H 6250 5550 50  0001 C CNN
 F 3 "http://www.ti.com/lit/ds/symlink/tl061.pdf" H 6350 5650 50  0001 C CNN
 	4    6300 5450
@@
 F 0 "U7" H 4650 2650 50  0000 L CNN
 F 1 "TL064" H 4600 2750 50  0000 L CNN
-F 2 "Package_DIP:DIP-14_W10.16mm_LongPads" H 4500 3050 50  0001 C CNN
+F 2 "Package_DIP:DIP-14_W7.62mm_Socket_LongPads" H 4500 3050 50  0001 C CNN
 F 3 "http://www.ti.com/lit/ds/symlink/tl061.pdf" H 4600 3150 50  0001 C CNN
 	5    4550 2950

Commit message: pcb reducido listo falta revisar
Parts:
- R2: footprint Resistor_THT:R_Axial_DIN0207_L6.3mm_D2.5mm_P7.62mm_Horizontal -> Resistor_THT:R_Axial_DIN0207_L6.3mm_D2.5mm_P10.16mm_Horizontal
Changed lines of the file:
@@
 F 0 "R7" V 3400 3050 50  0000 C CNN
 F 1 "1K" V 3300 3050 50  0000 C CNN
-F 2 "Resistor_THT:R_Axial_DIN0207_L6.3mm_D2.5mm_P7.62mm_Horizontal" V 3130 3050 50  0001 C CNN
+F 2 "Resistor_THT:R_Axial_DIN0207_L6.3mm_D2.5mm_P10.16mm_Horizontal" V 3130 3050 50  0001 C CNN
 F 3 "~" H 3200 3050 50  0001 C CNN
 	1    3200 3050
@@
 Entry Wire Line
 	2300 12550 2400 12450
-Wire Wire Line
-	6850 5450 6850 5050
 Wire Wire Line
 	6850 5050 5750 5050
@@
 Wire Wire Line
 	4550 6400 5350 6400
+Wire Wire Line
+	6850 5450 6850 5050
 $EndSCHEMATC

Commit message: calculos resistencias dac
Parts:
- R1, R2, R27: value 1K -> 10K
- R26: value 10K -> 8.2K
- R8: value 4K7 -> 5K6
- RV5: value R_POT -> 1K
Other:
- note added: "Salida DAC uC de 0 a 3.3V\nSalida módulo amplificador:\n0V = VEE (-5V)\n1.5V = 0V\n3.3V = VCC (5V)"
- note removed: "Salida DAC uC de 0 a 3V\nSalida módulo amplificador:\n0V = VEE (-5V)\n1.5V = 0V\n3V = VCC (5V)"
Changed lines of the file:
@@
 AR Path="/6013BA2D/5F8A81B2" Ref="R7"  Part="1"
 F 0 "R7" V 3400 3050 50  0000 C CNN
-F 1 "1K" V 3300 3050 50  0000 C CNN
+F 1 "10K" V 3300 3050 50  0000 C CNN
 F 2 "Resistor_THT:R_Axial_DIN0207_L6.3mm_D2.5mm_P10.16mm_Horizontal" V 3130 3050 50  0001 C CNN
 F 3 "~" H 3200 3050 50  0001 C CNN
@@
 AR Path="/6013BA2D/5F8A5925" Ref="R6"  Part="1"
 F 0 "R6" V 2993 2850 50  0000 C CNN
-F 1 "1K" V 3084 2850 50  0000 C CNN
+F 1 "10K" V 3084 2850 50  0000 C CNN
 F 2 "Resistor_THT:R_Axial_DIN0207_L6.3mm_D2.5mm_P7.62mm_Horizontal" V 3130 2850 50  0001 C CNN
 F 3 "~" H 3200 2850 50  0001 C CNN
@@
 	5750 5050 5750 5350
 Text Notes 2200 2700 0    50   ~ 0
-Salida DAC uC de 0 a 3V\nSalida módulo amplificador:\n0V = VEE (-5V)\n1.5V = 0V\n3V = VCC (5V)
+Salida DAC uC de 0 a 3.3V\nSalida módulo amplificador:\n0V = VEE (-5V)\n1.5V = 0V\n3.3V = VCC (5V)
 Text Notes 1400 7050 0    50   ~ 0
 Salida electrodo: VEE<0<VCC\nEntrada ADC: 0 a 5V (eventualmente 0 a 3.3V)
@@
 	4650 2450 4700 2450
 $Comp
-L salida_dac-rescue:R_POT-Device RV5
-U 1 1 5F9C3DAC
-P 4850 2450
-F 0 "RV5" V 4734 2450 50  0000 C CNN
-F 1 "R_POT" V 4641 2450 50  0000 C CNN
-F 2 "Potentiometer_THT:Potentiometer_Bourns_3266Y_Vertical" H 4850 2450 50  0001 C CNN
-F 3 "~" H 4850 2450 50  0001 C CNN
-	1    4850 2450
-	0    -1   -1   0
-$EndComp
-$Comp
 L salida_dac-rescue:R-Device R8
 U 1 1 5F8A592F
@@
 AR Path="/6013BA2D/5F8A592F" Ref="R13"  Part="1"
 F 0 "R13" V 4293 2450 50  0000 C CNN
-F 1 "4K7" V 4384 2450 50  0000 C CNN
+F 1 "5K6" V 4384 2450 50  0000 C CNN
 F 2 "Resistor_THT:R_Axial_DIN0207_L6.3mm_D2.5mm_P7.62mm_Horizontal" V 4430 2450 50  0001 C CNN
 F 3 "~" H 4500 2450 50  0001 C CNN
@@
 AR Path="/6013BA2D/605448B2" Ref="R26"  Part="1"
 F 0 "R26" V 2443 3500 50  0000 C CNN
-F 1 "10K" V 2534 3500 50  0000 C CNN
+F 1 "8.2K" V 2534 3500 50  0000 C CNN
 F 2 "Resistor_THT:R_Axial_DIN0207_L6.3mm_D2.5mm_P7.62mm_Horizontal" V 2580 3500 50  0001 C CNN
 F 3 "~" H 2650 3500 50  0001 C CNN
@@
 AR Path="/6013BA2D/605448BD" Ref="R27"  Part="1"
 F 0 "R27" V 3243 3500 50  0000 C CNN
-F 1 "1K" V 3334 3500 50  0000 C CNN
+F 1 "10K" V 3334 3500 50  0000 C CNN
 F 2 "Resistor_THT:R_Axial_DIN0207_L6.3mm_D2.5mm_P7.62mm_Horizontal" V 3380 3500 50  0001 C CNN
 F 3 "~" H 3450 3500 50  0001 C CNN
@@
 Wire Wire Line
 	6850 5450 6850 5050
+$Comp
+L salida_dac-rescue:R_POT-Device RV5
+U 1 1 5F9C3DAC
+P 4850 2450
+F 0 "RV5" V 4734 2450 50  0000 C CNN
+F 1 "1K" V 4641 2450 50  0000 C CNN
+F 2 "Potentiometer_THT:Potentiometer_Bourns_3266Y_Vertical" H 4850 2450 50  0001 C CNN
+F 3 "~" H 4850 2450 50  0001 C CNN
+	1    4850 2450
+	0    -1   -1   0
+$EndComp
 $EndSCHEMATC

Commit message: modificaciones R
Parts:
- R4: value 4K7 -> 10K
- R8, R9: value 1K -> 10K
Changed lines of the file:
@@
 VIN
-$Comp
-L salida_dac-rescue:R-Device R9
-U 1 1 5F9506D4
-P 4400 6200
-AR Path="/5F9506D4" Ref="R9"  Part="1"
-AR Path="/5F899696/5F9506D4" Ref="R14"  Part="1"
-AR Path="/6013BA2D/5F9506D4" Ref="R14"  Part="1"
-F 0 "R14" V 4193 6200 50  0000 C CNN
-F 1 "1K" V 4284 6200 50  0000 C CNN
-F 2 "Resistor_THT:R_Axial_DIN0207_L6.3mm_D2.5mm_P7.62mm_Horizontal" V 4330 6200 50  0001 C CNN
-F 3 "~" H 4400 6200 50  0001 C CNN
-	1    4400 6200
-	0    -1   1    0
-$EndComp
 $Comp
 L salida_dac-rescue:R-Device R4
@@
 AR Path="/6013BA2D/5F9506DA" Ref="R9"  Part="1"
 F 0 "R9" V 2993 5750 50  0000 C CNN
-F 1 "4K7" V 3084 5750 50  0000 C CNN
+F 1 "10K" V 3084 5750 50  0000 C CNN
 F 2 "Resistor_THT:R_Axial_DIN0207_L6.3mm_D2.5mm_P7.62mm_Horizontal" V 3130 5750 50  0001 C CNN
 F 3 "~" H 3200 5750 50  0001 C CNN
@@
 P 4400 6400
 F 0 "R8" V 4500 6400 50  0000 C CNN
-F 1 "1K" V 4600 6400 50  0000 C CNN
+F 1 "10K" V 4600 6400 50  0000 C CNN
 F 2 "Resistor_THT:R_Axial_DIN0207_L6.3mm_D2.5mm_P7.62mm_Horizontal" V 4330 6400 50  0001 C CNN
 F 3 "~" H 4400 6400 50  0001 C CNN
@@
 	0    -1   -1   0
 $EndComp
+$Comp
+L salida_dac-rescue:R-Device R9
+U 1 1 5F9506D4
+P 4400 6200
+AR Path="/5F9506D4" Ref="R9"  Part="1"
+AR Path="/5F899696/5F9506D4" Ref="R14"  Part="1"
+AR Path="/6013BA2D/5F9506D4" Ref="R14"  Part="1"
+F 0 "R14" V 4193 6200 50  0000 C CNN
+F 1 "10K" V 4284 6200 50  0000 C CNN
+F 2 "Resistor_THT:R_Axial_DIN0207_L6.3mm_D2.5mm_P7.62mm_Horizontal" V 4330 6200 50  0001 C CNN
+F 3 "~" H 4400 6200 50  0001 C CNN
+	1    4400 6200
+	0    -1   1    0
+$EndComp
 $EndSCHEMATC

Commit message: agregado lo de Hernan y fixeado el kicad pcb
Parts:
- R13: renamed from R8; value 5K6 -> 6K8
- R17: renamed from R16; value 1K -> 10K
- R18: renamed from R10; value 1K -> 10K
- R9: renamed from R4; value 10K -> 4K7
- renumbered R27 to R10, R9 to R11, R8 to R12, R10 to R14, R11 to R15, R13 to R16, R17 to R19, R18 to R20, R26 to R6, R1 to R7, R2 to R8, RV12 to RV2, RV2 to RV3, RV5 to RV4, RV6 to RV5, RV8 to RV6, RV10 to RV7, U7 to U5
